Commit message: add Neato file

File: neato_node2/urdf/neato.urdf (robot description, URDF)
Before this commit: robot neato_standalone, 1 links, 0 joints
Links:
- added link base_footprint
- added link base_laser_link, mass 0.0001
- added link camera_link, mass 1e-5; collision box size=0.05 0.05 0.05; visual box size=0.05 0.05 0.05
- added link caster_back_left_link, mass 0.01; collision cylinder length=0.0176 radius=0.01
- added link caster_back_right_link, mass 0.01; collision cylinder length=0.0176 radius=0.01
- added link caster_front_left_link, mass 0.01; collision cylinder length=0.0176 radius=0.01
- added link caster_front_right_link, mass 0.01; collision cylinder length=0.0176 radius=0.01
- added link cliff_sensor_left_link, mass 0.0001
- added link cliff_sensor_right_link, mass 0.0001
- added link imu_link, mass 0.001
- added link wheel_left_link, mass 0.01; collision cylinder length=0.0206 radius=0.035; visual mesh filename=package://neato_node2/wheel.dae
- added link wheel_right_link, mass 0.01; collision cylinder length=0.0206 radius=0.035; visual mesh filename=package://neato_node2/wheel.dae
Joints:
- added joint base_joint: type fixed, parent base_footprint, child base_link, origin xyz=0 0 0 rpy=0 0 0
- added joint camera_joint: type fixed, parent base_link, child camera_link, origin xyz=-0.1 0 0.25 rpy=0 0 0, axis 0 1 0
- added joint caster_back_left_joint: type fixed, parent base_link, child caster_back_left_link, origin xyz=-0.11 0.09 0 rpy=1.5707963267948966 0 0
- added joint caster_back_right_joint: type fixed, parent base_link, child caster_back_right_link, origin xyz=-0.11 -0.09 0 rpy=1.5707963267948966 0 0
- added joint caster_front_left_joint: type fixed, parent base_link, child caster_front_left_link, origin xyz=0.08 0.075 0 rpy=1.5707963267948966 0 0
- added joint caster_front_right_joint: type fixed, parent base_link, child caster_front_right_link, origin xyz=0.08 -0.075 0 rpy=1.5707963267948966 0 0
- added joint cliff_sensor_left_joint: type fixed, parent base_link, child cliff_sensor_left_link, origin xyz=0.11 0.145 0 rpy=0 1.5707963267948966 0
- added joint cliff_sensor_right_joint: type fixed, parent base_link, child cliff_sensor_right_link, origin xyz=0.11 -0.145 0 rpy=0 1.5707963267948966 0
- added joint imu_joint: type fixed, parent base_link, child imu_link, origin xyz=0 0 0 rpy=0 0 0, axis 0 1 0
- added joint laser_joint: type fixed, parent base_link, child base_laser_link, origin xyz=-0.084 0 0.166 rpy=0 0 3.141592653589793
- added joint wheel_left_joint: type continuous, parent base_link, child wheel_left_link, origin xyz=0.00 0.1175 0.0250 rpy=0 0 0, axis 0 1 0
- added joint wheel_right_joint: type continuous, parent base_link, child wheel_right_link, origin xyz=0.00 -0.1175 0.0250 rpy=0 0 0, axis 0 1 0
