Commit message: very basic Neato simulator

File: neato2_interfaces/urdf/neato.urdf (robot description, URDF)
Before this commit: robot neato_standalone, 13 links, 12 joints
Links:
- link base_link: geometry collision box size=0.16 0.3 0.06; collision cylinder length=0.06 radius=0.15
- link camera_link: geometry collision box size=0.05 0.05 0.05
- link wheel_left_link: geometry collision cylinder length=0.0206 radius=0.035; visual mesh filename=package://neato2_interfaces/models/neato/meshes/wheel.dae
- link wheel_right_link: geometry collision cylinder length=0.0206 radius=0.035; visual mesh filename=package://neato2_interfaces/models/neato/meshes/wheel.dae
